File: pcb/untitled.kicad_sch (KiCad schematic)
At the start: 15 parts, among them IC3 AD844ANZ, IC5 FOD814SD, U2 REF192GSZ

Commit message: Updated resistor values
updated two resistor values to coincide with changes made to my circuit. R12 and R21 are the names.
Changed lines of the file:
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@@
   (junction (at 44.45 64.77) (diameter 0) (color 0 0 0 0)
+  )
+  (junction (at 24.13 64.77) (diameter 0) (color 0 0 0 0)
   )
   (junction (at 193.04 127) (diameter 0) (color 0 0 0 0)
@@
     (stroke (width 0) (type default))
   )
+  (wire (pts (xy 24.13 57.15) (xy 24.13 64.77))
+    (stroke (width 0) (type default))
+  )
   (wire (pts (xy 184.15 118.11) (xy 184.15 125.73))
     (stroke (width 0) (type default))
@@
         )
       )
+    )
+  )
+  (symbol (lib_id "power:PWR_FLAG") (at 24.13 57.15 0) (unit 1)
+    (in_bom yes) (on_board yes) (dnp no) (fields_autoplaced)
+    (property "Reference" "#FLG05" (at 24.13 55.245 0)
+      (effects (font (size 1.27 1.27)) hide)
+    )
+    (property "Value" "PWR_FLAG" (at 24.13 52.07 0)
+      (effects (font (size 1.27 1.27)))
+    )
+    (property "Footprint" "" (at 24.13 57.15 0)
+      (effects (font (size 1.27 1.27)) hide)
+    )
+    (property "Datasheet" "~" (at 24.13 57.15 0)
+      (effects (font (size 1.27 1.27)) hide)
+    )
+    (pin "1")
+    (instances
+      (project "mcu_integration"
+        (path "/c0210bc3-f67f-47d8-a34e-f002a728adb2/f1afd235-040c-4b54-9b6d-8df613af2103"
+          (reference "#FLG05") (unit 1)
+        )
+      )
