File: pcb/mcu_integration.kicad_pcb (KiCad board)
At the start: 4 copper layers, 100 x 100 mm, 104 parts, among them IC1 TL7660IDGKR, IC10 AD844_OPAMP_MEL, IC2 TL081IDT, IC3 FOD814_OPTO_NOSHD, IC4 UA78M33CDCYG3, IC5 FOD814_OPTO_MEL, IC6 AD844_OPAMP_AL, IC7 FOD814_OPTO_AL, IC8 AD844_OPAMP_NOSHD, J1 Micro_SD_Card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

Commit message: add names to project
Routing:
- net ADC1_IN0_SINE: track 257.1 -> 255.0 mm
Other:
- board text added: "*"
- board text added: "CUBICS Analog IC Shielding Payload Karim A., Evan C., Matthew H. REV B March 6th, 2024"
Changed lines of the file:
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@@
         (effects (font (size 1 1) (thickness 0.15)))
     )
-    (fp_text user "*" (at -1.61925 2.54 unlocked) (layer "F.SilkS")
-        (effects (font (size 1 1) (thickness 0.15)))
-    )
-    (fp_text user "*" (at -2.54 2.54) (layer "F.SilkS")
+    (fp_text user "*" (at -1.65 -1.8) (layer "F.SilkS")
         (effects (font (size 1 1) (thickness 0.15)))
     )
@@
     (effects (font (size 1 1) (thickness 0.15)) (justify left bottom))
   )
+  (gr_text "*" (at 126.7 86.4) (layer "F.SilkS")
+    (effects (font (size 1 1) (thickness 0.15)) (justify left bottom))
+  )
   (gr_text "NOSHD" (at 116.4 123.8) (layer "F.SilkS")
     (effects (font (size 1 1) (thickness 0.15)) (justify left bottom))
@@
     (effects (font (size 1 1) (thickness 0.15)) (justify left bottom))
   )
+  (gr_text "CUBICS Analog IC Shielding Payload\nKarim A., Evan C., Matthew H.\nREV B\nMarch 6th, 2024" (at 94.4 79.4) (layer "F.SilkS")
+    (effects (font (size 1 1) (thickness 0.15)) (justify left bottom))
+  )
   (gr_text "E_NOSHD" (at 116.4 103.5) (layer "F.SilkS")
     (effects (font (size 1 1) (thickness 0.15)) (justify left bottom))
@@
   (segment (start 105.7 107.48995) (end 113.01005 114.8) (width 0.3) (layer "B.Cu") (net 189))
   (segment (start 91 82.8) (end 89.125 84.675) (width 0.25) (layer "F.Cu") (net 190))
-  (segment (start 92.5 118.73) (end 93.1375 118.73) (width 0.3) (layer "F.Cu") (net 190))
+  (segment (start 110.4 114.8) (end 110.4 123.425) (width 0.3) (layer "F.Cu") (net 190))
   (segment (start 101.09 108) (end 101.09 108.69) (width 0.3) (layer "F.Cu") (net 190))
-  (segment (start 110.4 114.8) (end 110.4 124.6) (width 0.3) (layer "F.Cu") (net 190))
   (segment (start 109.4 136.42) (end 109.4 142.4) (width 0.3) (layer "F.Cu") (net 190))
   (segment (start 167.434634 114.175) (end 175.88 122.620366) (width 0.3) (layer "F.Cu") (net 190))
   (segment (start 112.2 128.02) (end 115 130.82) (width 0.3) (layer "F.Cu") (net 190))
-  (segment (start 104.774 110.6) (end 103 110.6) (width 0.3) (layer "F.Cu") (net 190))
   (segment (start 127.325 93.25) (end 128.75 93.25) (width 0.3) (layer "F.Cu") (net 190))
   (segment (start 90.45072 108.445) (end 91.155 108.445) (width 0.25) (layer "F.Cu") (net 190))
   (segment (start 109.4 142.4) (end 108.07 143.73) (width 0.3) (layer "F.Cu") (net 190))
-  (segment (start 112.2 113) (end 110.4 114.8) (width 0.3) (layer "F.Cu") (net 190))
   (segment (start 101.09 108.69) (end 103 110.6) (width 0.3) (layer "F.Cu") (net 190))
-  (segment (start 110.4 116.226) (end 104.774 110.6) (width 0.3) (layer "F.Cu") (net 190))
   (segment (start 115 130.82) (end 109.523 136.297) (width 0.3) (layer "F.Cu") (net 190))
+  (segment (start 104.774 110.6) (end 103 110.6) (width 0.3) (layer "F.Cu") (net 190))
   (segment (start 112.2 113) (end 112.2 128.02) (width 0.3) (layer "F.Cu") (net 190))
   (segment (start 89.125 84.675) (end 89.125 107.11928) (width 0.25) (layer "F.Cu") (net 190))
+  (segment (start 110.4 123.425) (end 110.4 116.226) (width 0.3) (layer "F.Cu") (net 190))
+  (segment (start 110.4 123.425) (end 109.5 124.325) (width 0.3) (layer "F.Cu") (net 190))
+  (segment (start 93.1375 118.73) (end 98.7325 124.325) (width 0.3) (layer "F.Cu") (net 190))
   (segment (start 145.6 114) (end 145.775 114.175) (width 0.3) (layer "F.Cu") (net 190))
   (segment (start 175.88 122.620366) (end 175.88 127.13) (width 0.3) (layer "F.Cu") (net 190))
   (segment (start 145.775 114.175) (end 167.434634 114.175) (width 0.3) (layer "F.Cu") (net 190))
-  (segment (start 110.4 124.6) (end 110.4 116.226) (width 0.3) (layer "F.Cu") (net 190))
-  (segment (start 98.7325 124.325) (end 110.125 124.325) (width 0.3) (layer "F.Cu") (net 190))
+  (segment (start 98.7325 124.325) (end 109.5 124.325) (width 0.3) (layer "F.Cu") (net 190))
+  (segment (start 110.4 116.226) (end 104.774 110.6) (width 0.3) (layer "F.Cu") (net 190))
   (segment (start 92.8495 131.385) (end 92.212 131.385) (width 0.3) (layer "F.Cu") (net 190))
-  (segment (start 93.1375 118.73) (end 98.7325 124.325) (width 0.3) (layer "F.Cu") (net 190))
+  (segment (start 92.5 118.73) (end 93.1375 118.73) (width 0.3) (layer "F.Cu") (net 190))
   (segment (start 128.75 93.25) (end 129 93) (width 0.3) (layer "F.Cu") (net 190))
   (segment (start 109.523 136.297) (end 97.7615 136.297) (width 0.3) (layer "F.Cu") (net 190))
   (segment (start 89.125 107.11928) (end 90.45072 108.445) (width 0.25) (layer "F.Cu") (net 190))
   (segment (start 94.6 110.6) (end 91.8 107.8) (width 0.3) (layer "F.Cu") (net 190))
+  (segment (start 112.2 113) (end 110.4 114.8) (width 0.3) (layer "F.Cu") (net 190))
   (segment (start 103 110.6) (end 94.6 110.6) (width 0.3) (layer "F.Cu") (net 190))
   (segment (start 97.7615 136.297) (end 92.8495 131.385) (width 0.3) (layer "F.Cu") (net 190))
   (segment (start 115 130.82) (end 109.4 136.42) (width 0.3) (layer "F.Cu") (net 190))
   (segment (start 91.155 108.445) (end 91.8 107.8) (width 0.25) (layer "F.Cu") (net 190))
-  (segment (start 110.125 124.325) (end 110.4 124.6) (width 0.3) (layer "F.Cu") (net 190))
   (segment (start 175.88 127.13) (end 175.26 127.75) (width 0.3) (layer "F.Cu") (net 190))
   (segment (start 108.07 143.73) (end 105.576 143.73) (width 0.3) (layer "F.Cu") (net 190))
